Commit message: Multiple Camera of Octocopter model added

File: urdf/octorotor_base.urdf.xacro (robot description, xacro)
@@ -1,5 +1,4 @@
 <?xml version="1.0"?>
 <robot xmlns:xacro="http://ros.org/wiki/xacro">
-  <xacro:include filename="$(find hector_sensors_description)/urdf/sonar_sensor.urdf.xacro" />
   <xacro:property name="pi" value="3.1415926535897931" />
   <!-- Main quadrotor link -->
@@ -24,8 +23,4 @@
       </collision>
     </link>
-    <!-- Sonar height sensor -->
-    <xacro:sonar_sensor name="sonar" parent="base_link" ros_topic="sonar_height" update_rate="10" min_range="0.03" max_range="3.0" field_of_view="${40*pi/180}" ray_count="3">
-      <origin xyz="-0.16 0.0 -0.012" rpy="0 ${90*pi/180} 0"/>
-    </xacro:sonar_sensor>
   </xacro:macro>
 </robot>

File: urdf/octorotor_with_asus.urdf.xacro (robot description, xacro)
@@ -10,7 +10,10 @@
     <xacro:quadrotor_base_macro />
     <!-- Asus Xiton Live Pro -->
-    <xacro:include filename="$(find hector_sensors_description)/urdf/asus_camera.urdf.xacro" />
+    <xacro:include filename="$(find swarm_stereo)/urdf/asus_camera.urdf.xacro" />
     <xacro:asus_camera name="camera" parent="base_link">
-      <origin xyz="0.1 0.0 -0.03" rpy="0 ${M_PI/9} 0"/>
+      <origin xyz="0.0 0.1 -0.03" rpy="0 ${M_PI/9} 0"/>
+    </xacro:asus_camera>
+    <xacro:asus_camera name="camera1" parent="base_link">
+      <origin xyz="0.0 -0.1 -0.03" rpy="0 ${M_PI/9} 0"/>
     </xacro:asus_camera>
 </robot>
